File: board.sch (EAGLE design)
At the start: 6 parts, among them J1 POWER_JACK, J2 POWER_JACK, J3 POWER_JACK, J4 POWER_JACK, J5 POWER_JACK, J6 POWER_JACK

Commit message: git ignore, add cooper fills (for testing)
Connections:
- net N$1 renamed GND
- net N$2 renamed VCC
Changed lines of the file:
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@@
 </busses>
 <nets>
-<net name="N$1" class="0">
+<net name="GND" class="0">
 <segment>
 <pinref part="J1" gate="G$1" pin="PWR"/>
@@
 <wire x1="58.42" y1="2.54" x2="58.42" y2="15.24" width="0.1524" layer="91"/>
 <junction x="58.42" y="15.24"/>
+<label x="58.42" y="66.04" size="1.778" layer="95"/>
 </segment>
 </net>
-<net name="N$2" class="0">
+<net name="VCC" class="0">
 <segment>
 <pinref part="J1" gate="G$1" pin="GNDBREAK"/>
@@
 <wire x1="48.26" y1="0" x2="48.26" y2="12.7" width="0.1524" layer="91"/>
 <junction x="48.26" y="12.7"/>
+<label x="48.26" y="48.26" size="1.778" layer="95"/>
 </segment>
 </net>
